File: hardware/orio-carrier/conv12_5.kicad_sch (KiCad schematic)
At the start: 33 parts, among them J3 12 V aux / lights, U3 TPS54360B, U4 TPS54360B

Commit message: Make every footprint resolve against KiCad's own libraries
Six of the 28 footprint references were names chosen by inspection that
don't exist, so "Update PCB from Schematic" would have failed on them.
Checked against a real KiCad 10 install and fixed:

  L_Bourns-SRN6045TA          -> L_Bourns_SRN6045TA (hyphen vs underscore)
  L_Bourns_SRP1265A           -> L_Bourns_SRP1245A (same SRP12xx 12.5mm land)
  VQFN-24-1EP_4x4mm...        -> HVQFN-24-1EP_4x4mm..._ThermalVias
  SOIC-8-1EP...EP2.29x3.0mm   -> ...EP2.29x3mm_ThermalVias
  SolderWirePad_1x02_P5.08mm  -> SolderWire-4sqmm_1x02_P12mm (12 AWG, XT60)

The thermal-via variants are the right call for the LM5145 and both
TPS54360B stages regardless -- they dissipate, and the vias were going to
be added by hand otherwise.

The B0505S-1WR3 has no answer in KiCad: no MORNSUN library exists and the
part is a SIP-4 whose pins are not a 2.54 mm inline row. Substituting a
Murata converter with different pin spacing would be a dead board that
looks fine, so it is a declared placeholder in FP_PLACEHOLDER instead,
reported on every run alongside the unverified pin tables.

generate.py now resolves all 28 against a local KiCad install when it
finds one, and stays silent when it doesn't so the generator still runs
on a machine with only Python.

Co-Authored-By: Claude Opus 5 <noreply@anthropic.com>
Parts:
- L2, L3: footprint Inductor_SMD:L_Bourns-SRN6045TA -> Inductor_SMD:L_Bourns_SRN6045TA
- U3, U4: footprint Package_SO:SOIC-8-1EP_3.9x4.9mm_P1.27mm_EP2.29x3.0mm -> Package_SO:SOIC-8-1EP_3.9x4.9mm_P1.27mm_EP2.29x3mm_ThermalVias
Changed lines of the file:
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@@
     (property "Reference" "U3" (at 66.04 38.1 0) (effects (font (size 1.27 1.27)) (justify left)))
     (property "Value" "TPS54360B" (at 66.04 58.42 0) (effects (font (size 1.27 1.27)) (justify left)))
-    (property "Footprint" "Package_SO:SOIC-8-1EP_3.9x4.9mm_P1.27mm_EP2.29x3.0mm" (at 66.04 48.26 0) (effects (font (size 1.27 1.27)) (hide yes)))
+    (property "Footprint" "Package_SO:SOIC-8-1EP_3.9x4.9mm_P1.27mm_EP2.29x3mm_ThermalVias" (at 66.04 48.26 0) (effects (font (size 1.27 1.27)) (hide yes)))
     (pin "1")
     (pin "2")
@@
     (property "Reference" "L2" (at 66.04 99.06 0) (effects (font (size 1.27 1.27)) (justify left)))
     (property "Value" "15uH 4A" (at 66.04 109.22 0) (effects (font (size 1.27 1.27)) (justify left)))
-    (property "Footprint" "Inductor_SMD:L_Bourns-SRN6045TA" (at 66.04 104.14 0) (effects (font (size 1.27 1.27)) (hide yes)))
+    (property "Footprint" "Inductor_SMD:L_Bourns_SRN6045TA" (at 66.04 104.14 0) (effects (font (size 1.27 1.27)) (hide yes)))
     (pin "1")
     (pin "2")
@@
     (property "Reference" "U4" (at 66.04 246.38 0) (effects (font (size 1.27 1.27)) (justify left)))
     (property "Value" "TPS54360B" (at 66.04 266.7 0) (effects (font (size 1.27 1.27)) (justify left)))
-    (property "Footprint" "Package_SO:SOIC-8-1EP_3.9x4.9mm_P1.27mm_EP2.29x3.0mm" (at 66.04 256.54 0) (effects (font (size 1.27 1.27)) (hide yes)))
+    (property "Footprint" "Package_SO:SOIC-8-1EP_3.9x4.9mm_P1.27mm_EP2.29x3mm_ThermalVias" (at 66.04 256.54 0) (effects (font (size 1.27 1.27)) (hide yes)))
     (pin "1")
     (pin "2")
@@
     (property "Reference" "L3" (at 66.04 307.34 0) (effects (font (size 1.27 1.27)) (justify left)))
     (property "Value" "6.8uH 5A" (at 66.04 317.5 0) (effects (font (size 1.27 1.27)) (justify left)))
-    (property "Footprint" "Inductor_SMD:L_Bourns-SRN6045TA" (at 66.04 312.42 0) (effects (font (size 1.27 1.27)) (hide yes)))
-    (pin "1")
-    (pin "2")
+    (property "Footprint" "Inductor_SMD:L_Bourns_SRN6045TA" (at 66.04 312.42 0) (effects (font (size 1.27 1.27)) (hide yes)))
+    (pin "1")
+    (pin "2")
