File: hardware/orio-carrier/drivetrain.kicad_sch (KiCad schematic)
At the start: 33 parts, among them J20 FSESC L, J21 FSESC R, J22 E-stop (NC), U10 ISO7721DR, U11 AP2112K-3.3, U12 AP2112K-3.3, U9 ISO7721DR

Commit message: Make every footprint resolve against KiCad's own libraries
Six of the 28 footprint references were names chosen by inspection that
don't exist, so "Update PCB from Schematic" would have failed on them.
Checked against a real KiCad 10 install and fixed:

  L_Bourns-SRN6045TA          -> L_Bourns_SRN6045TA (hyphen vs underscore)
  L_Bourns_SRP1265A           -> L_Bourns_SRP1245A (same SRP12xx 12.5mm land)
  VQFN-24-1EP_4x4mm...        -> HVQFN-24-1EP_4x4mm..._ThermalVias
  SOIC-8-1EP...EP2.29x3.0mm   -> ...EP2.29x3mm_ThermalVias
  SolderWirePad_1x02_P5.08mm  -> SolderWire-4sqmm_1x02_P12mm (12 AWG, XT60)

The thermal-via variants are the right call for the LM5145 and both
TPS54360B stages regardless -- they dissipate, and the vias were going to
be added by hand otherwise.

The B0505S-1WR3 has no answer in KiCad: no MORNSUN library exists and the
part is a SIP-4 whose pins are not a 2.54 mm inline row. Substituting a
Murata converter with different pin spacing would be a dead board that
looks fine, so it is a declared placeholder in FP_PLACEHOLDER instead,
reported on every run alongside the unverified pin tables.

generate.py now resolves all 28 against a local KiCad install when it
finds one, and stays silent when it doesn't so the generator still runs
on a machine with only Python.

Co-Authored-By: Claude Opus 5 <noreply@anthropic.com>
Parts:
- PS1, PS2: footprint Converter_DCDC:Converter_DCDC_MORNSUN_B0505S-1WR3_SIP -> Connector_PinHeader_2.54mm:PinHeader_1x04_P2.54mm_Vertical
Changed lines of the file:
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@@
     (property "Reference" "PS1" (at 66.04 204.47 0) (effects (font (size 1.27 1.27)) (justify left)))
     (property "Value" "B0505S-1WR3" (at 66.04 217.17 0) (effects (font (size 1.27 1.27)) (justify left)))
-    (property "Footprint" "Converter_DCDC:Converter_DCDC_MORNSUN_B0505S-1WR3_SIP" (at 66.04 210.82 0) (effects (font (size 1.27 1.27)) (hide yes)))
+    (property "Footprint" "Connector_PinHeader_2.54mm:PinHeader_1x04_P2.54mm_Vertical" (at 66.04 210.82 0) (effects (font (size 1.27 1.27)) (hide yes)))
     (pin "1")
     (pin "2")
@@
     (property "Reference" "PS2" (at 66.04 433.07 0) (effects (font (size 1.27 1.27)) (justify left)))
     (property "Value" "B0505S-1WR3" (at 66.04 445.77 0) (effects (font (size 1.27 1.27)) (justify left)))
-    (property "Footprint" "Converter_DCDC:Converter_DCDC_MORNSUN_B0505S-1WR3_SIP" (at 66.04 439.42 0) (effects (font (size 1.27 1.27)) (hide yes)))
-    (pin "1")
-    (pin "2")
+    (property "Footprint" "Connector_PinHeader_2.54mm:PinHeader_1x04_P2.54mm_Vertical" (at 66.04 439.42 0) (effects (font (size 1.27 1.27)) (hide yes)))
+    (pin "1")
+    (pin "2")
